Commit message: URDF and launch file changes

File: src/vox/description/camera.xacro (robot description, xacro)
@@ -20,26 +20,3 @@
 	</joint>
 	<link name="camera_link_optical"></link>
-	<gazebo reference="camera_link">
-		<material>Gazebo/Blue</material>
-		<sensor name="camera" type="camera">
-			<pose> 0 0 0 0 0 0 </pose>
-			<visualize>true</visualize>
-			<update_rate>10</update_rate>
-			<camera>
-				<horizontal_fov>1.15192</horizontal_fov>
-				<image>
-					<format>R8G8B8</format>
-					<width>640</width>
-					<height>480</height>
-				</image>
-				<clip>
-					<near>0.05</near>
-					<far>8.0</far>
-				</clip>
-			</camera>
-			<plugin name="camera_controller" filename="libgazebo_ros_camera.so">
-				<frame_name>camera_link_optical</frame_name>
-			</plugin>
-		</sensor>
-	</gazebo>
 </robot>

File: src/vox/description/laser.xacro (robot description, xacro)
@@ -28,33 +28,3 @@
         </inertial>
 	</link>
-	<gazebo reference="laser_frame">
-		<material>Gazebo/Blue</material>
-		<sensor name="laser" type="ray">
-			<pose> 0 0 0 0 0 0 </pose>
-			<visualize>false</visualize>
-			<update_rate>10</update_rate>
-			<ray>
-				<scan>
-					<horizontal>
-						<samples>360</samples>
-						<resolution>1</resolution>
-						<min_angle>-3.14</min_angle>
-						<max_angle>3.14</max_angle>
-					</horizontal>
-				</scan>
-				<range>
-					<min>0.3</min>
-					<max>12</max>
-					<resolution>0.01</resolution>
-				</range>
-			</ray>
-			<plugin name="laser_controller" filename="libgazebo_ros_ray_sensor.so">
-				<ros>
-					<argument>~/out:=scan</argument>
-				</ros>
-				<output_type>sensor_msgs/LaserScan</output_type>
-				<frame_name>laser_frame</frame_name>
-			</plugin>
-		</sensor>
-	</gazebo>
 </robot>

File: src/vox/description/robot.urdf.xacro (robot description, xacro)
@@ -1,12 +1,6 @@
 <?xml version="1.0"?>
 <robot xmlns:xacro="http://www.ros.org/wiki/xacro" name="vox">
-	<xacro:arg name="use_ros2_control" default="false"/>
 	<xacro:include filename="robot_core.xacro"/>
-	<xacro:if value="$(arg use_ros2_control)">
-		<xacro:include filename="ros2_control.xacro"/>
-	</xacro:if>
-	<xacro:unless value="$(arg use_ros2_control)">
-		<xacro:include filename="gazebo_controls.xacro"/>
-	</xacro:unless>
+	<xacro:include filename="ros2_control.xacro"/>
 	<xacro:include filename="laser.xacro"/>
 	<xacro:include filename="camera.xacro"/>

File: src/vox/description/robot_core.xacro (robot description, xacro)
@@ -2,7 +2,5 @@
 <robot xmlns:xacro="http://www.ros.org/wiki/xacro">
     <xacro:include filename="colors.xacro"/>
-    <!-- BASE LINK -->
     <link name="base_link"></link>
-    <!-- BASE FOOTPRINT LINK -->
     <joint name="base_footprint_joint" type="fixed">
         <parent link="base_link"/>
@@ -11,5 +9,4 @@
     </joint>
     <link name="base_footprint"></link>
-    <!-- CHASSIS LINK -->
     <joint name="chassis_joint" type="fixed">
         <parent link="base_link"/>
@@ -40,7 +37,4 @@
         </inertial>
     </link>
-    <gazebo reference="chassis">
-        <material>Gazebo/White</material>
-    </gazebo>
     <joint name="front_left_wheel_joint" type="continuous">
         <parent link="chassis"/>
@@ -58,5 +52,4 @@
         <collision>
             <geometry>
-                <!-- <cylinder radius="0.06" length="0.06"/> -->
                 <sphere radius="0.06"/>
             </geometry>
@@ -72,7 +65,4 @@
         </inertial>
     </link>
-    <gazebo reference="front_left_wheel">
-        <material>Gazebo/Blue</material>
-    </gazebo>
     <joint name="front_right_wheel_joint" type="continuous">
         <parent link="chassis"/>
@@ -90,5 +80,4 @@
         <collision>
             <geometry>
-                <!-- <cylinder radius="0.06" length="0.06"/> -->
                 <sphere radius="0.06"/>
             </geometry>
@@ -104,7 +93,4 @@
         </inertial>
     </link>
-    <gazebo reference="front_right_wheel">
-        <material>Gazebo/Blue</material>
-    </gazebo>
     <joint name="back_left_wheel_joint" type="continuous">
         <parent link="chassis"/>
@@ -122,5 +108,4 @@
         <collision>
             <geometry>
-                <!-- <cylinder radius="0.06" length="0.06"/> -->
                 <sphere radius="0.06"/>
             </geometry>
@@ -136,7 +121,4 @@
         </inertial>
     </link>
-    <gazebo reference="back_left_wheel">
-        <material>Gazebo/Blue</material>
-    </gazebo>
     <joint name="back_right_wheel_joint" type="continuous">
         <parent link="chassis"/>
@@ -154,5 +136,4 @@
         <collision>
             <geometry>
-                <!-- <cylinder radius="0.06" length="0.06"/> -->
                 <sphere radius="0.06"/>
             </geometry>
@@ -168,6 +149,3 @@
         </inertial>
     </link>
-    <gazebo reference="back_right_wheel">
-        <material>Gazebo/Blue</material>
-    </gazebo>
 </robot>
